File: V3S_SBC/Clock.kicad_sch (KiCad schematic)
At the start: 4 parts, among them Y1 24Mhz

Commit message: Add files via upload
Parts:
- removed C17, C18: 12pF, symbol Device:C
- removed R12: 1M, symbol Device:R
- removed Y1: 24Mhz, symbol Device:Crystal
- added C20, C21: 12pF, symbol Device:C
- added R20: 1M, symbol Device:R
- added Y2: 32.768kHz, symbol Device:Crystal
Connections:
- net GND: now also C20.2, C21.2
- new net 32kHz IN: C20.1, R20.1, Y2.1
- new net 32kHz OUT: C21.1, R20.2, Y2.2
