File: V3S_SBC/MicroSD.kicad_sch (KiCad schematic)
At the start: 10 parts, among them J2 Micro_SD_Card_Det1, U3 USBLC6-2SC6

Commit message: Add files via upload
Parts:
- removed U3: USBLC6-2SC6, Package_TO_SOT_SMD:SOT-23-6, symbol Power_Protection:USBLC6-2SC6
Changed lines of the file:
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@@
-	)
-	(symbol
-		(lib_id "Power_Protection:USBLC6-2SC6")
-		(at 97.79 113.03 0)
-		(unit 1)
-		(body_style 1)
-		(exclude_from_sim no)
-		(in_bom yes)
-		(on_board yes)
-		(in_pos_files yes)
-		(dnp no)
-		(fields_autoplaced yes)
-		(property "Reference" "U3"
-			(at 99.4411 105.41 0)
-			(show_name no)
-			(do_not_autoplace no)
-			(effects
-				(font
-					(size 1.27 1.27)
-				)
-				(justify left)
-			)
-		)
-		(property "Value" "USBLC6-2SC6"
-			(at 99.4411 107.95 0)
-			(show_name no)
-			(do_not_autoplace no)
-			(effects
-				(font
-					(size 1.27 1.27)
-				)
-				(justify left)
-			)
-		)
-		(property "Footprint" "Package_TO_SOT_SMD:SOT-23-6"
-			(at 99.06 119.38 0)
-			(hide yes)
-			(show_name no)
-			(do_not_autoplace no)
-			(effects
-				(font
-					(size 1.27 1.27)
-					(italic yes)
-				)
-				(justify left)
-			)
-		)
-		(property "Datasheet" "https://www.st.com/resource/en/datasheet/usblc6-2.pdf"
-			(at 99.06 121.285 0)
-			(hide yes)
-			(show_name no)
-			(do_not_autoplace no)
-			(effects
-				(font
-					(size 1.27 1.27)
-				)
-				(justify left)
-			)
-		)
-		(property "Description" "Very low capacitance ESD protection diode, 2 data-line, SOT-23-6"
-			(at 97.79 113.03 0)
-			(hide yes)
-			(show_name no)
-			(do_not_autoplace no)
-			(effects
-				(font
-					(size 1.27 1.27)
-				)
-			)
-		)
-		(pin "3"
-		)
-		(pin "1"
-		)
-		(pin "2"
-		)
-		(pin "4"
-		)
-		(pin "6"
-		)
-		(pin "5"
-		)
-		(instances
-			(project "V3S_SBC"
-				(path "/d510d0d2-5c6c-421d-aef5-78001d333beb/f5dc1a3d-d3ca-43a7-9896-1d9481fd90ba"
-					(reference "U3")
-					(unit 1)
-				)
-			)
-		)
 	)
 	(symbol

Commit message: Add files via upload
Changed lines of the file:
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@@
-	)
-	(junction
-		(at 128.27 85.09)
-		(diameter 0)
-		(color 0 0 0 0)
 	)
 	(junction
@@
 	(wire
 		(pts
-			(xy 120.65 85.09) (xy 128.27 85.09)
-		)
-		(stroke
-			(width 0)
-			(type default)
-		)
-	)
-	(wire
-		(pts
 			(xy 116.84 77.47) (xy 116.84 80.01)
 		)
@@
 	(wire
 		(pts
-			(xy 128.27 85.09) (xy 138.43 85.09)
+			(xy 120.65 85.09) (xy 138.43 85.09)
 		)
 		(stroke
@@
 		(pts
 			(xy 128.27 80.01) (xy 138.43 80.01)
-		)
-		(stroke
-			(width 0)
-			(type default)
-		)
-	)
-	(wire
-		(pts
-			(xy 128.27 83.82) (xy 128.27 85.09)
 		)
 		(stroke
@@
 			)
 			(justify right)
-		)
-	)
-	(hierarchical_label "VCC"
-		(shape bidirectional)
-		(at 128.27 83.82 0)
-		(effects
-			(font
-				(size 1.27 1.27)
-			)
-			(justify left)
 		)
 	)
@@
 		(instances
 			(project "V3S_SBC"
-				(path "/d510d0d2-5c6c-421d-aef5-78001d333beb/f5dc1a3d-d3ca-43a7-9896-1d9481fd90ba"
+				(path "/d510d0d2-5c6c-421d-aef5-78001d333beb/752bb6c1-a34c-41f3-9a33-185e78878f4a"
 					(reference "R15")
 					(unit 1)
@@
 		(instances
 			(project "V3S_SBC"
-				(path "/d510d0d2-5c6c-421d-aef5-78001d333beb/f5dc1a3d-d3ca-43a7-9896-1d9481fd90ba"
+				(path "/d510d0d2-5c6c-421d-aef5-78001d333beb/752bb6c1-a34c-41f3-9a33-185e78878f4a"
 					(reference "R17")
 					(unit 1)
@@
 		(instances
 			(project "V3S_SBC"
-				(path "/d510d0d2-5c6c-421d-aef5-78001d333beb/f5dc1a3d-d3ca-43a7-9896-1d9481fd90ba"
+				(path "/d510d0d2-5c6c-421d-aef5-78001d333beb/752bb6c1-a34c-41f3-9a33-185e78878f4a"
 					(reference "R13")
 					(unit 1)
@@
 		(instances
 			(project "V3S_SBC"
-				(path "/d510d0d2-5c6c-421d-aef5-78001d333beb/f5dc1a3d-d3ca-43a7-9896-1d9481fd90ba"
+				(path "/d510d0d2-5c6c-421d-aef5-78001d333beb/752bb6c1-a34c-41f3-9a33-185e78878f4a"
 					(reference "R19")
 					(unit 1)
@@
 		(instances
 			(project "V3S_SBC"
-				(path "/d510d0d2-5c6c-421d-aef5-78001d333beb/f5dc1a3d-d3ca-43a7-9896-1d9481fd90ba"
+				(path "/d510d0d2-5c6c-421d-aef5-78001d333beb/752bb6c1-a34c-41f3-9a33-185e78878f4a"
 					(reference "J2")
 					(unit 1)
@@
 		(instances
 			(project "V3S_SBC"
-				(path "/d510d0d2-5c6c-421d-aef5-78001d333beb/f5dc1a3d-d3ca-43a7-9896-1d9481fd90ba"
+				(path "/d510d0d2-5c6c-421d-aef5-78001d333beb/752bb6c1-a34c-41f3-9a33-185e78878f4a"
 					(reference "R16")
 					(unit 1)
@@
 		(instances
 			(project "V3S_SBC"
-				(path "/d510d0d2-5c6c-421d-aef5-78001d333beb/f5dc1a3d-d3ca-43a7-9896-1d9481fd90ba"
+				(path "/d510d0d2-5c6c-421d-aef5-78001d333beb/752bb6c1-a34c-41f3-9a33-185e78878f4a"
 					(reference "R14")
 					(unit 1)
@@
 		(instances
 			(project "V3S_SBC"
-				(path "/d510d0d2-5c6c-421d-aef5-78001d333beb/f5dc1a3d-d3ca-43a7-9896-1d9481fd90ba"
+				(path "/d510d0d2-5c6c-421d-aef5-78001d333beb/752bb6c1-a34c-41f3-9a33-185e78878f4a"
 					(reference "R18")
 					(unit 1)
@@
 		(instances
 			(project "V3S_SBC"
-				(path "/d510d0d2-5c6c-421d-aef5-78001d333beb/f5dc1a3d-d3ca-43a7-9896-1d9481fd90ba"
+				(path "/d510d0d2-5c6c-421d-aef5-78001d333beb/752bb6c1-a34c-41f3-9a33-185e78878f4a"
 					(reference "C19")
 					(unit 1)
