File: V3S_SBC/V3S_SBC.kicad_sch (KiCad schematic)
At the start: 1 part, among them U1 V3S

Commit message: Add files via upload
Other:
- added sheet Clock (Clock.kicad_sch)
- added sheet MicroSD (MicroSD.kicad_sch)
Changed lines of the file:
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@@
+	)
+	(sheet
+		(at 226.06 150.495)
+		(size 22.86 12.7)
+		(exclude_from_sim no)
+		(in_bom yes)
+		(on_board yes)
+		(dnp no)
+		(fields_autoplaced yes)
+		(stroke
+			(width 0.1524)
+			(type solid)
+		)
+		(fill
+			(color 0 0 0 0)
+		)
+		(property "Sheetname" "Clock"
+			(at 226.06 149.7834 0)
+			(show_name no)
+			(do_not_autoplace no)
+			(effects
+				(font
+					(size 1.27 1.27)
+				)
+				(justify left bottom)
+			)
+		)
+		(property "Sheetfile" "Clock.kicad_sch"
+			(at 226.06 163.7796 0)
+			(show_name no)
+			(do_not_autoplace no)
+			(effects
+				(font
+					(size 1.27 1.27)
+				)
+				(justify left top)
+			)
+		)
+		(instances
+			(project "V3S_SBC"
+				(path "/d510d0d2-5c6c-421d-aef5-78001d333beb"
+					(page "3")
+				)
+			)
+		)
 	)
 	(sheet
@@
 				)
 			)
+		)
+	)
+	(sheet
+		(at 229.235 105.41)
+		(size 38.735 19.685)
+		(exclude_from_sim no)
+		(in_bom yes)
+		(on_board yes)
+		(dnp no)
+		(fields_autoplaced yes)
+		(stroke
+			(width 0.1524)
+			(type solid)
+		)
+		(fill
+			(color 0 0 0 0)
+		)
+		(property "Sheetname" "MicroSD"
+			(at 229.235 104.6984 0)
+			(show_name no)
+			(do_not_autoplace no)
+			(effects
+				(font
+					(size 1.27 1.27)
+				)
+				(justify left bottom)
+			)
+		)
+		(property "Sheetfile" "MicroSD.kicad_sch"
+			(at 229.235 125.6796 0)
+			(show_name no)
+			(do_not_autoplace no)
+			(effects
+				(font
+					(size 1.27 1.27)
+				)
+				(justify left top)
+			)
+		)
+		(instances
+			(project "V3S_SBC"
+				(path "/d510d0d2-5c6c-421d-aef5-78001d333beb"
+					(page "4")
+				)
+			)

Commit message: Add files via upload
Parts:
- added C20, C21, C22, C23, C26, C27, C28, C29, C30, C31: 0.1uF, symbol Device:C
- added J3: Conn_01x03_Pin, symbol Connector:Conn_01x03_Pin
Connections:
- net Power Module/USB-DM: now reaches U1.110 (USB-DM)
- net Power Module/USB-DP: now reaches U1.111 (USB-DP)
- net +3.3V_IO: now reaches U1.12 (VCC-PE0)
- net +3.3V_IO: now also U1.127 (VCC-IO1), U1.29 (VCC-PE1), C26.1, C27.1
- net +1.2V_Core: now reaches U1.20 (VDD-CPU3)
- net +1.2V_Core: now also U1.21 (VDD-CPU2), U1.25 (VDD-CPU1), U1.26 (VDD-CPU0), U1.38 (VDD-CPU4), U1.47 (VDD-CPU5), U1.51 (VDD-CPU6), U1.56 (VDD-CPU7), C20.1, C21.1, C22.1, C23.1, C28.1, C29.1, C30.1, C31.1
- net at U1.48 (PB8/TWI1_SCK/UART0_TX/PB_EINT8): now also J3.1 (Pin_1)
- net at U1.49 (PB9/TWI1_SDA/UART0_RX/PB_EINT9): now also J3.2 (Pin_2)
- net Clock/24MHz OUT: now reaches U1.74 (X24MOUT)
- net Clock/24MHz IN: now reaches U1.75 (X24MIN)
- new net GND: C20.2, C21.2, C22.2, C23.2, C26.2, C27.2, C28.2, C29.2, C30.2, C31.2, J3.3 (Pin_3)
Other:
- sheet Clock ports: added 24MHz IN, 24MHz OUT, GND; removed none
- sheet Power Module ports: added +1.2V_Core, +3.0V_AVcc, +3.3V_IO, +5V, GND, USB-DM, USB-DP; removed none

Commit message: Add files via upload
Parts:
- removed C20, C21, C22, C23, C26, C27, C28, C29, C30, C31: 0.1uF, symbol Device:C
- added C32, C33, C34, C35, C36, C37, C38, C39, C40, C41, C42, C43, C44, C45, C46, C47, C48, C49, C50, C51: 0.1uF, symbol Device:C
- added R12: 10kOhm, symbol Device:R
Connections:
- net +1.2V_Core: now also U1.108 (VDD-SYS1), U1.126 (VDD-SYS2), U1.19 (VDD-SYS3), U1.58 (VDD-SYS4), U1.64 (VDD-SYS5), U1.80 (VDD-SYS0), C32.1, C33.1, C34.1, C35.1, C36.1, C37.1, C38.1, C39.1, C40.1, C41.1, C42.1, C43.1, C44.1, C45.1
- net +3.3V_IO: now also U1.104 (VCC-IO0), U1.109 (VCC-USB), U1.50 (VCC-IO3), U1.57 (VCC-IO2), C46.1, C47.1, C48.1, C49.1, C50.1, R12.1; no longer U1.12 (VCC-PE0), U1.29 (VCC-PE1)
- net GND: now also C32.2, C33.2, C34.2, C35.2, C36.2, C37.2, C38.2, C39.2, C40.2, C41.2, C42.2, C43.2, C44.2, C45.2, C46.2, C47.2, C48.2, C49.2, C50.2, C51.1
- net MicroSD/Detect: now reaches U1.100 (PF6)
- net MicroSD/DATA2: now reaches U1.101 (F5/SDC0_D2/JTAG_CK1)
- net MicroSD/DATA3: now reaches U1.102 (PF4/SDC0_D3/UART0_RX)
- net MicroSD/CMD: now reaches U1.103 (PF3/SDC0_CMD/JTAG_DO1)
- net MicroSD/CLK: now reaches U1.105 (PF2/SDC0_CLK/UART0_TX)
- net MicroSD/DATA0: now reaches U1.106 (PF1/SDC0_D0/JTAG_DI1)
- net MicroSD/DATA1: now reaches U1.107 (PF0/SDC0_D1/JTAG_MS1)
- net Clock32k/32kHz OUT: now reaches U1.95 (X32KOUT)
- net Clock32k/32kHz IN: now reaches U1.96 (X32KIN)
- net at U1.99 (RESET): now also C51.2, R12.2
Other:
- added sheet Clock32k (Clock.kicad_sch)
- added sheet LCD (LCD.kicad_sch)
- sheet MicroSD ports: added +3.3v, CLK, CMD, DATA0, DATA1, DATA2, DATA3, Detect, GND; removed none
- moved on the sheet: J3

Commit message: Add files via upload
Parts:
- added J10: Port 4, symbol Connector:USB_A
- added J11, J8: Port2, symbol Connector:USB_A
- added J6: UART2, symbol Connector:Conn_01x03_Pin
- added J7: UART1, symbol Connector:Conn_01x03_Pin
- added J9: Port3, symbol Connector:USB_A
- J3: value Conn_01x03_Pin -> UART0
Connections:
- net +5V: now also J10.1 (VBUS), J11.1 (VBUS), J8.1 (VBUS), J9.1 (VBUS)
- net GND: now also J10.4 (GND), J10.SH (Shield), J11.4 (GND), J11.SH (Shield), J6.3 (Pin_3), J7.3 (Pin_3), J8.4 (GND), J8.SH (Shield), J9.4 (GND), J9.SH (Shield)
- net LCD_CLK: now reaches U1.37 (PE0/CSI_PCLK/LCD_CLK)
- net at U1.39 (PB0/UART2_TX/PB_EINT0): now also J6.1 (Pin_1)
- net at U1.40 (PB1/UART2_RX/PB_EINT1): now also J6.2 (Pin_2)
- net at U1.8 (PE22/CSI_SDA/TWI1_SDA/UART1_RX): now also J7.2 (Pin_2)
- net at U1.9 (PE21/CSI_SCK/TWI1_SCK/UART1_TX): now also J7.1 (Pin_1)
- net Power Module/USB-DM renamed USB/USB-DM
- net Power Module/USB-DP renamed USB/USB-DP
- new net Port1-DM: J11.2 (D-)
- new net Port1-DP: J11.3 (D+)
- new net Port2-DM: J8.2 (D-)
- new net Port2-DP: J8.3 (D+)
- new net Port3-DM: J9.2 (D-)
- new net Port3-DP: J9.3 (D+)
- new net Port4-DM: J10.2 (D-)
- new net Port4-DP: J10.3 (D+)
Other:
- added sheet USB (USB.kicad_sch)
- sheet LCD ports: added GND, IO-VCC, LCD_CLK, PB5 CTP-INT, PB6 (IO_SCL), PB7 (IO_SDA), PD22 DISP, PE0, PE1, PE10, PE11, PE12, PE13, PE14, PE15, PE16, PE17, PE19 (LCD_DE), PE2, PE20 CTP-RST, PE3, PE4, PE5, PE6, PE7, PE8, PE9; removed none
- sheet Power Module ports: added none; removed USB-DM, USB-DP
- note added: "TRG"
- note removed: "JLC"
